File: PCB_kicad/alpha_pro_micro.sch (KiCad schematic (older format))
At the start: 59 parts, among them J1 Conn_01x03, K1 KEYSW, K10 KEYSW, K11 KEYSW, K12 KEYSW, K13 KEYSW, K14 KEYSW, K15 KEYSW, K16 KEYSW, K17 KEYSW, K18 KEYSW, K19 KEYSW, K2 KEYSW, K20 KEYSW, K21 KEYSW, K22 KEYSW, K23 KEYSW, K24 KEYSW, K25 KEYSW, K26 KEYSW, K27 KEYSW, K28 KEYSW, K3 KEYSW, K4 KEYSW, K5 KEYSW, K6 KEYSW, K7 KEYSW, K8 KEYSW, K9 KEYSW, SW1 SW_Push, U1 ProMicro

Commit message: Begin PCB rework
Parts:
- K1, K10, K11, K12, K13, K14, K15, K16, K17, K18, K19, K2, K20, K21, K22, K23, K24, K26, K27, K28, K3, K4, K5, K6, K7, K8, K9: footprint keebio-parts:MX-Alps-Choc-1U-NoLED -> MX_Alps_Hybrid:MXOnly-1U-NoLED
- K25: footprint keebio-parts:MX-Alps-Choc-2U-StabFlip -> MX_Alps_Hybrid:MXOnly-2U-ReversedStabilizers-NoLED
Connections:
- net col0: now also K1.1, K11.1, K21.1; no longer K1.2, K11.2, K21.2
- net col1: now also K12.1, K2.1, K22.1; no longer K12.2, K2.2, K22.2
- net col2: now also K13.1, K23.1, K3.1; no longer K13.2, K23.2, K3.2
- net col3: now also K14.1, K24.1, K4.1; no longer K14.2, K24.2, K4.2
- net col4: now also K15.1, K5.1; no longer K15.2, K5.2
- net col5: now also K16.1, K6.1; no longer K16.2, K6.2
- net col6: now also K17.1, K7.1; no longer K17.2, K7.2
- net col7: now also K18.1, K26.1, K8.1; no longer K18.2, K26.2, K8.2
- net col8: now also K19.1, K27.1, K9.1; no longer K19.2, K27.2, K9.2
- net col9: now also K10.1, K20.1, K28.1; no longer K10.2, K20.2, K28.2
- net at D2.2 (A): now also K2.2; no longer K2.1
- net at D1.2 (A): now also K1.2; no longer K1.1
- net at D3.2 (A): now also K3.2; no longer K3.1
- net at D11.2 (A): now also K11.2; no longer K11.1
- net at D12.2 (A): now also K12.2; no longer K12.1
- net at D13.2 (A): now also K13.2; no longer K13.1
- net at D4.2 (A): now also K4.2; no longer K4.1
- net at D14.2 (A): now also K14.2; no longer K14.1
- net at D15.2 (A): now also K15.2; no longer K15.1
- net at D16.2 (A): now also K16.2; no longer K16.1
- net at D5.2 (A): now also K5.2; no longer K5.1
- net at D6.2 (A): now also K6.2; no longer K6.1
- net at D21.2 (A): now also K21.2; no longer K21.1
- net at D22.2 (A): now also K22.2; no longer K22.1
- net at D23.2 (A): now also K23.2; no longer K23.1
- net at D24.2 (A): now also K24.2; no longer K24.1
- net at D27.2 (A): now also K27.2; no longer K27.1
- net at D7.2 (A): now also K7.2; no longer K7.1
- net at D8.2 (A): now also K8.2; no longer K8.1
- net at D9.2 (A): now also K9.2; no longer K9.1
- net at D10.2 (A): now also K10.2; no longer K10.1
- net at D17.2 (A): now also K17.2; no longer K17.1
- net at D18.2 (A): now also K18.2; no longer K18.1
- net at D19.2 (A): now also K19.2; no longer K19.1
- net at D20.2 (A): now also K20.2; no longer K20.1
- net at D26.2 (A): now also K26.2; no longer K26.1
- net at D28.2 (A): now also K28.2; no longer K28.1
Changed lines of the file:
@@
 EESchema Schematic File Version 4
-LIBS:alpha_pro_micro-cache
-EELAYER 29 0
+EELAYER 30 0
 EELAYER END
 $Descr A4 11693 8268
@@
 F 0 "K11" H 1150 4400 60  0000 C CNN
 F 1 "KEYSW" H 1200 4300 60  0001 C CNN
-F 2 "keebio-parts:MX-Alps-Choc-1U-NoLED" H 1200 4400 60  0001 C CNN
+F 2 "MX_Alps_Hybrid:MXOnly-1U-NoLED" H 1200 4400 60  0001 C CNN
 F 3 "" H 1200 4400 60  0000 C CNN
 	1    1200 4400
-	-1   0    0    -1
+	1    0    0    -1
 $EndComp
 $Comp
@@
 F 0 "K12" H 2100 4400 60  0000 C CNN
 F 1 "KEYSW" H 2150 4300 60  0001 C CNN
-F 2 "keebio-parts:MX-Alps-Choc-1U-NoLED" H 2150 4400 60  0001 C CNN
+F 2 "MX_Alps_Hybrid:MXOnly-1U-NoLED" H 2150 4400 60  0001 C CNN
 F 3 "" H 2150 4400 60  0000 C CNN
 	1    2150 4400
-	-1   0    0    -1
+	1    0    0    -1
 $EndComp
 $Comp
@@
 F 0 "K13" H 3050 4450 60  0000 C CNN
 F 1 "KEYSW" H 3100 4350 60  0001 C CNN
-F 2 "keebio-parts:MX-Alps-Choc-1U-NoLED" H 3100 4450 60  0001 C CNN
+F 2 "MX_Alps_Hybrid:MXOnly-1U-NoLED" H 3100 4450 60  0001 C CNN
 F 3 "" H 3100 4450 60  0000 C CNN
 	1    3100 4450
-	-1   0    0    -1
+	1    0    0    -1
 $EndComp
 $Comp
@@
 F 0 "K14" H 4150 4450 60  0000 C CNN
 F 1 "KEYSW" H 4200 4350 60  0001 C CNN
-F 2 "keebio-parts:MX-Alps-Choc-1U-NoLED" H 4200 4450 60  0001 C CNN
+F 2 "MX_Alps_Hybrid:MXOnly-1U-NoLED" H 4200 4450 60  0001 C CNN
 F 3 "" H 4200 4450 60  0000 C CNN
 	1    4200 4450
-	-1   0    0    -1
+	1    0    0    -1
 $EndComp
 $Comp
@@
 F 0 "K15" H 5050 4450 60  0000 C CNN
 F 1 "KEYSW" H 5100 4350 60  0001 C CNN
-F 2 "keebio-parts:MX-Alps-Choc-1U-NoLED" H 5100 4450 60  0001 C CNN
+F 2 "MX_Alps_Hybrid:MXOnly-1U-NoLED" H 5100 4450 60  0001 C CNN
 F 3 "" H 5100 4450 60  0000 C CNN
 	1    5100 4450
-	-1   0    0    -1
+	1    0    0    -1
 $EndComp
 $Comp
@@
 F 0 "K16" H 5900 4450 60  0000 C CNN
 F 1 "KEYSW" H 5950 4350 60  0001 C CNN
-F 2 "keebio-parts:MX-Alps-Choc-1U-NoLED" H 5950 4450 60  0001 C CNN
+F 2 "MX_Alps_Hybrid:MXOnly-1U-NoLED" H 5950 4450 60  0001 C CNN
 F 3 "" H 5950 4450 60  0000 C CNN
 	1    5950 4450
-	-1   0    0    -1
+	1    0    0    -1
 $EndComp
 $Comp
@@
 F 0 "K21" H 1750 5150 60  0000 C CNN
 F 1 "KEYSW" H 1800 5050 60  0001 C CNN
-F 2 "keebio-parts:MX-Alps-Choc-1U-NoLED" H 1800 5150 60  0001 C CNN
+F 2 "MX_Alps_Hybrid:MXOnly-1U-NoLED" H 1800 5150 60  0001 C CNN
 F 3 "" H 1800 5150 60  0000 C CNN
 	1    1800 5150
-	-1   0    0    -1
+	1    0    0    -1
 $EndComp
 $Comp
@@
 F 0 "K22" H 2650 5150 60  0000 C CNN
 F 1 "KEYSW" H 2700 5050 60  0001 C CNN
-F 2 "keebio-parts:MX-Alps-Choc-1U-NoLED" H 2700 5150 60  0001 C CNN
+F 2 "MX_Alps_Hybrid:MXOnly-1U-NoLED" H 2700 5150 60  0001 C CNN
 F 3 "" H 2700 5150 60  0000 C CNN
 	1    2700 5150
-	-1   0    0    -1
+	1    0    0    -1
 $EndComp
 $Comp
@@
 F 0 "K23" H 3600 5150 60  0000 C CNN
 F 1 "KEYSW" H 3650 5050 60  0001 C CNN
-F 2 "keebio-parts:MX-Alps-Choc-1U-NoLED" H 3650 5150 60  0001 C CNN
+F 2 "MX_Alps_Hybrid:MXOnly-1U-NoLED" H 3650 5150 60  0001 C CNN
 F 3 "" H 3650 5150 60  0000 C CNN
 	1    3650 5150
-	-1   0    0    -1
+	1    0    0    -1
 $EndComp
 $Comp
@@
 F 0 "K24" H 4650 5150 60  0000 C CNN
 F 1 "KEYSW" H 4700 5050 60  0001 C CNN
-F 2 "keebio-parts:MX-Alps-Choc-1U-NoLED" H 4700 5150 60  0001 C CNN
+F 2 "MX_Alps_Hybrid:MXOnly-1U-NoLED" H 4700 5150 60  0001 C CNN
 F 3 "" H 4700 5150 60  0000 C CNN
 	1    4700 5150
-	-1   0    0    -1
+	1    0    0    -1
 $EndComp
 $Comp
@@
 F 0 "K25" H 5900 5150 60  0000 C CNN
 F 1 "KEYSW" H 5950 5050 60  0001 C CNN
-F 2 "keebio-parts:MX-Alps-Choc-2U-StabFlip" H 5950 5150 60  0001 C CNN
+F 2 "MX_Alps_Hybrid:MXOnly-2U-ReversedStabilizers-NoLED" H 5950 5150 60  0001 C CNN
 F 3 "" H 5950 5150 60  0000 C CNN
 	1    5950 5150
@@
 F 0 "K27" H 8500 5150 60  0000 C CNN
 F 1 "KEYSW" H 8550 5050 60  0001 C CNN
-F 2 "keebio-parts:MX-Alps-Choc-1U-NoLED" H 8550 5150 60  0001 C CNN
+F 2 "MX_Alps_Hybrid:MXOnly-1U-NoLED" H 8550 5150 60  0001 C CNN
 F 3 "" H 8550 5150 60  0000 C CNN
 	1    8550 5150
-	-1   0    0    -1
+	1    0    0    -1
 $EndComp
 $Comp
@@
 F 0 "K9" H 9050 3700 60  0000 C CNN
 F 1 "KEYSW" H 9100 3600 60  0001 C CNN
-F 2 "keebio-parts:MX-Alps-Choc-1U-NoLED" H 9100 3700 60  0001 C CNN
+F 2 "MX_Alps_Hybrid:MXOnly-1U-NoLED" H 9100 3700 60  0001 C CNN
 F 3 "" H 9100 3700 60  0000 C CNN
 	1    9100 3700
-	-1   0    0    -1
+	1    0    0    -1
 $EndComp
 $Comp
@@
 F 0 "K10" H 10000 3700 60  0000 C CNN
 F 1 "KEYSW" H 10050 3600 60  0001 C CNN
-F 2 "keebio-parts:MX-Alps-Choc-1U-NoLED" H 10050 3700 60  0001 C CNN
+F 2 "MX_Alps_Hybrid:MXOnly-1U-NoLED" H 10050 3700 60  0001 C CNN
 F 3 "" H 10050 3700 60  0000 C CNN
 	1    10050 3700
-	-1   0    0    -1
+	1    0    0    -1
 $EndComp
 $Comp
@@
 F 0 "K17" H 7100 4500 60  0000 C CNN
 F 1 "KEYSW" H 7150 4400 60  0001 C CNN
-F 2 "keebio-parts:MX-Alps-Choc-1U-NoLED" H 7150 4500 60  0001 C CNN
+F 2 "MX_Alps_Hybrid:MXOnly-1U-NoLED" H 7150 4500 60  0001 C CNN
 F 3 "" H 7150 4500 60  0000 C CNN
 	1    7150 4500
-	-1   0    0    -1
+	1    0    0    -1
 $EndComp
 $Comp
@@
 F 0 "K18" H 8050 4500 60  0000 C CNN
 F 1 "KEYSW" H 8100 4400 60  0001 C CNN
-F 2 "keebio-parts:MX-Alps-Choc-1U-NoLED" H 8100 4500 60  0001 C CNN
+F 2 "MX_Alps_Hybrid:MXOnly-1U-NoLED" H 8100 4500 60  0001 C CNN
 F 3 "" H 8100 4500 60  0000 C CNN
 	1    8100 4500
-	-1   0    0    -1
+	1    0    0    -1
 $EndComp
 $Comp
@@
 F 0 "K19" H 9050 4500 60  0000 C CNN
 F 1 "KEYSW" H 9100 4400 60  0001 C CNN
-F 2 "keebio-parts:MX-Alps-Choc-1U-NoLED" H 9100 4500 60  0001 C CNN
+F 2 "MX_Alps_Hybrid:MXOnly-1U-NoLED" H 9100 4500 60  0001 C CNN
 F 3 "" H 9100 4500 60  0000 C CNN
 	1    9100 4500
-	-1   0    0    -1
+	1    0    0    -1
 $EndComp
 $Comp
@@
 F 0 "K20" H 10000 4500 60  0000 C CNN
 F 1 "KEYSW" H 10050 4400 60  0001 C CNN
-F 2 "keebio-parts:MX-Alps-Choc-1U-NoLED" H 10050 4500 60  0001 C CNN
+F 2 "MX_Alps_Hybrid:MXOnly-1U-NoLED" H 10050 4500 60  0001 C CNN
 F 3 "" H 10050 4500 60  0000 C CNN
 	1    10050 4500
-	-1   0    0    -1
+	1    0    0    -1
 $EndComp
 $Comp
@@
 F 0 "K26" H 7400 5150 60  0000 C CNN
 F 1 "KEYSW" H 7450 5050 60  0001 C CNN
-F 2 "keebio-parts:MX-Alps-Choc-1U-NoLED" H 7450 5150 60  0001 C CNN
+F 2 "MX_Alps_Hybrid:MXOnly-1U-NoLED" H 7450 5150 60  0001 C CNN
 F 3 "" H 7450 5150 60  0000 C CNN
 	1    7450 5150
-	-1   0    0    -1
+	1    0    0    -1
 $EndComp
 $Comp
@@
 F 0 "K28" H 9500 5150 60  0000 C CNN
 F 1 "KEYSW" H 9550 5050 60  0001 C CNN
-F 2 "keebio-parts:MX-Alps-Choc-1U-NoLED" H 9550 5150 60  0001 C CNN
+F 2 "MX_Alps_Hybrid:MXOnly-1U-NoLED" H 9550 5150 60  0001 C CNN
 F 3 "" H 9550 5150 60  0000 C CNN
 	1    9550 5150
-	-1   0    0    -1
+	1    0    0    -1
 $EndComp
 $Comp
@@
 F 0 "K8" H 8050 3700 60  0000 C CNN
 F 1 "KEYSW" H 8100 3600 60  0001 C CNN
-F 2 "keebio-parts:MX-Alps-Choc-1U-NoLED" H 8100 3700 60  0001 C CNN
+F 2 "MX_Alps_Hybrid:MXOnly-1U-NoLED" H 8100 3700 60  0001 C CNN
 F 3 "" H 8100 3700 60  0000 C CNN
 	1    8100 3700
-	-1   0    0    -1
+	1    0    0    -1
 $EndComp
 $Comp
@@
 F 0 "K7" H 7100 3700 60  0000 C CNN
 F 1 "KEYSW" H 7150 3600 60  0001 C CNN
-F 2 "keebio-parts:MX-Alps-Choc-1U-NoLED" H 7150 3700 60  0001 C CNN
+F 2 "MX_Alps_Hybrid:MXOnly-1U-NoLED" H 7150 3700 60  0001 C CNN
 F 3 "" H 7150 3700 60  0000 C CNN
 	1    7150 3700
-	-1   0    0    -1
+	1    0    0    -1
 $EndComp
 $Comp
@@
 F 0 "K6" H 6050 3700 60  0000 C CNN
 F 1 "KEYSW" H 6100 3600 60  0001 C CNN
-F 2 "keebio-parts:MX-Alps-Choc-1U-NoLED" H 6100 3700 60  0001 C CNN
+F 2 "MX_Alps_Hybrid:MXOnly-1U-NoLED" H 6100 3700 60  0001 C CNN
 F 3 "" H 6100 3700 60  0000 C CNN
 	1    6100 3700
-	-1   0    0    -1
+	1    0    0    -1
 $EndComp
 $Comp
@@
 F 0 "K5" H 5100 3700 60  0000 C CNN
 F 1 "KEYSW" H 5150 3600 60  0001 C CNN
-F 2 "keebio-parts:MX-Alps-Choc-1U-NoLED" H 5150 3700 60  0001 C CNN
+F 2 "MX_Alps_Hybrid:MXOnly-1U-NoLED" H 5150 3700 60  0001 C CNN
 F 3 "" H 5150 3700 60  0000 C CNN
 	1    5150 3700
-	-1   0    0    -1
+	1    0    0    -1
 $EndComp
 $Comp
@@
 F 0 "K4" H 4150 3650 60  0000 C CNN
 F 1 "KEYSW" H 4200 3550 60  0001 C CNN
-F 2 "keebio-parts:MX-Alps-Choc-1U-NoLED" H 4200 3650 60  0001 C CNN
+F 2 "MX_Alps_Hybrid:MXOnly-1U-NoLED" H 4200 3650 60  0001 C CNN
 F 3 "" H 4200 3650 60  0000 C CNN
 	1    4200 3650
-	-1   0    0    -1
+	1    0    0    -1
 $EndComp
 $Comp
@@
 F 0 "K3" H 3100 3650 60  0000 C CNN
 F 1 "KEYSW" H 3150 3550 60  0001 C CNN
-F 2 "keebio-parts:MX-Alps-Choc-1U-NoLED" H 3150 3650 60  0001 C CNN
+F 2 "MX_Alps_Hybrid:MXOnly-1U-NoLED" H 3150 3650 60  0001 C CNN
 F 3 "" H 3150 3650 60  0000 C CNN
 	1    3150 3650
-	-1   0    0    -1
+	1    0    0    -1
 $EndComp
 $Comp
@@
 F 0 "K2" H 2100 3650 60  0000 C CNN
 F 1 "KEYSW" H 2150 3550 60  0001 C CNN
-F 2 "keebio-parts:MX-Alps-Choc-1U-NoLED" H 2150 3650 60  0001 C CNN
+F 2 "MX_Alps_Hybrid:MXOnly-1U-NoLED" H 2150 3650 60  0001 C CNN
 F 3 "" H 2150 3650 60  0000 C CNN
 	1    2150 3650
-	-1   0    0    -1
+	1    0    0    -1
 $EndComp
 $Comp
@@
 F 0 "K1" H 1200 3650 60  0000 C CNN
 F 1 "KEYSW" H 1250 3550 60  0001 C CNN
-F 2 "keebio-parts:MX-Alps-Choc-1U-NoLED" H 1250 3650 60  0001 C CNN
+F 2 "MX_Alps_Hybrid:MXOnly-1U-NoLED" H 1250 3650 60  0001 C CNN
 F 3 "" H 1250 3650 60  0000 C CNN
 	1    1250 3650
-	-1   0    0    -1
-$EndComp
-Wire Wire Line
+	1    0    0    -1
+$EndComp
+Wire Wire Line
